File: Hardware/Bus_switch.kicad_sch (KiCad schematic)
At the start: 14 parts, among them U1 SN74CB3Q3384APW

Commit message: V1.1
Connections:
- net Chainbus.RX: now also U1.5 (1B2); no longer U1.2 (1B1)
- net Chainbus.TX: now also U1.2 (1B1); no longer U1.5 (1B2)
Other:
- note added: "ISSUE #2 FIX RX TX SWAP"
Changed lines of the file:
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@@
+		)
+	)
+	(text "ISSUE #2 FIX\nRX TX SWAP"
+		(exclude_from_sim no)
+		(at 99.822 71.628 0)
+		(effects
+			(font
+				(size 1.27 1.27)
+				(color 255 0 0 1)
+			)
 		)
 	)
@@
 	)
 	(bus_entry
-		(at 100.33 78.74)
+		(at 115.57 74.93)
 		(size -2.54 2.54)
 		(stroke
@@
 	)
 	(bus_entry
-		(at 100.33 81.28)
+		(at 115.57 77.47)
 		(size -2.54 2.54)
 		(stroke
@@
 		)
 	)
+	(wire
+		(pts
+			(xy 96.52 77.47) (xy 81.28 83.82)
+		)
+		(stroke
+			(width 0)
+			(type default)
+		)
+	)
 	(bus
 		(pts
@@
 		)
 	)
+	(polyline
+		(pts
+			(xy 92.964 77.978) (xy 94.234 77.724)
+		)
+		(stroke
+			(width 0)
+			(type solid)
+			(color 255 0 0 1)
+		)
+	)
 	(wire
 		(pts
@@
 	(wire
 		(pts
-			(xy 81.28 81.28) (xy 97.79 81.28)
+			(xy 96.52 77.47) (xy 113.03 77.47)
 		)
 		(stroke
@@
 		)
 	)
+	(polyline
+		(pts
+			(xy 92.456 76.2) (xy 92.964 77.978)
+		)
+		(stroke
+			(width 0)
+			(type solid)
+			(color 255 0 0 1)
+		)
+	)
 	(bus
 		(pts
@@
 	(bus
 		(pts
-			(xy 102.87 78.74) (xy 100.33 78.74)
+			(xy 118.11 74.93) (xy 115.57 74.93)
 		)
 		(stroke
@@
 	(wire
 		(pts
-			(xy 81.28 83.82) (xy 97.79 83.82)
+			(xy 96.52 80.01) (xy 113.03 80.01)
 		)
 		(stroke
@@
 	(wire
 		(pts
+			(xy 96.52 80.01) (xy 81.28 81.28)
+		)
+		(stroke
+			(width 0)
+			(type default)
+		)
+	)
+	(polyline
+		(pts
+			(xy 92.964 77.978) (xy 94.488 75.438)
+		)
+		(stroke
+			(width 0)
+			(type solid)
+			(color 255 0 0 1)
+		)
+	)
+	(wire
+		(pts
 			(xy 81.28 88.9) (xy 97.79 88.9)
 		)
@@
 	(bus
 		(pts
-			(xy 100.33 78.74) (xy 100.33 81.28)
+			(xy 115.57 74.93) (xy 115.57 77.47)
 		)
 		(stroke
@@
 	)
 	(label "Chainbus.TX"
-		(at 82.55 83.82 0)
+		(at 97.79 80.01 0)
 		(effects
 			(font
@@
 	)
 	(label "Chainbus.RX"
-		(at 82.55 81.28 0)
+		(at 97.79 77.47 0)
 		(effects
 			(font
@@
 	(hierarchical_label "Chainbus{UART}"
 		(shape bidirectional)
-		(at 102.87 78.74 0)
-		(effects
-			(font
+		(at 118.11 74.93 0)
+		(effects
+			(font
