File: Hardware/MMS3_hat_protocol.kicad_pcb (KiCad board)
At the start: 2 copper layers, 100 x 50 mm, 114 parts, among them J1 Chainbus in, J10 Conn_01x02_Pin, J11 Conn_01x04_Pin, J14 Conn_01x03_Pin, J15 Conn_01x04_Pin, J2 Chainbus Out, J3 Conn_01x02_Pin, J4 Conn_01x04_Pin, J5 Conn_01x03_Pin, J6 Conn_01x04_Pin, J7 Conn_01x06_Pin, J8 Conn_01x03_Pin, J9 Conn_01x04_Pin, U1 SN74CB3Q3384APW, U10 TXU0104PWR, U11 TXU0104PWR, U12 TXU0104PWR, U13 TCA9535PWR_C130204, U15 MAX13487EESA, U2 M24C64, U3 AMS1117, U4 TXU0104PWR, U5 TXU0104PWR, U6 MAX13487EESA, U8 TXU0104PWR, U9 PCA9306DCUR

Commit message: V1.1
Connections:
- U1 pad 2: /Chainbus.RX -> /Chainbus.TX
- U1 pad 5: /Chainbus.TX -> /Chainbus.RX
Routing:
- net /Chainbus.TX: track 59.2 -> 57.4 mm
- net /Chainbus.RX: track 47.7 -> 47.5 mm, vias 2 -> 3
